File: pcb/freq-counter.kicad_pcb (KiCad board)
At the start: 2 copper layers, 152.4 x 116.8 mm, 103 parts, among them J1 RPM on board, J10 Power_T1, J2 BNC, J3 RPM to Board, J4 Jack-DC, J5 Segments-Terminal0, J6 Digits-Terminal0, J7 Segments-Terminal1, J8 Digits-Terminal1, J9 Power_Terminal1, Q1 CSC388A, Q10 2SC1815, Q11 2SC1815, Q12 2SC1815, Q13 2SC1815, Q14 2SC1815, Q2 CSC388A, Q3 2SA1015, Q4 2SC1815, Q5 2SC1815, Q6 CSC388A, Q7 CSC388A, Q8 CSC388A, Q9 2SC1815, SW1 on/off, SW2 count up, SW3 toggle, SW4 SW_SIGNAL, U1 SN74HC02N, U2 ATTINY4313-PU(freq-counter), U3 EE-SX460, U4 74HC00, U5 74HC00, U6 74HC00, U7 7seg-2digit-ca, U8 7seg-2digit-ca, U9 7seg-2digit-ca, Y1 10MHz

Commit message: 4 layer に設定。In1.Cuがjumper layer，In2.Cuが電源layer。
Other:
- copper layers 2 -> 4
Changed lines of the file:
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@@
   (layers
     (0 F.Cu signal)
+    (1 In1.Cu jumper)
+    (2 In2.Cu power)
     (31 B.Cu signal)
-    (32 B.Adhes user)
     (33 F.Adhes user)
-    (34 B.Paste user)
     (35 F.Paste user)
-    (36 B.SilkS user)
     (37 F.SilkS user)
-    (38 B.Mask user)
     (39 F.Mask user)
     (40 Dwgs.User user)
@@
     (44 Edge.Cuts user)
     (45 Margin user)
-    (46 B.CrtYd user)
     (47 F.CrtYd user)
-    (48 B.Fab user)
     (49 F.Fab user)
   )

Commit message: 7SEG, LED, PUSH-BUTTON 等の入出力関係は上部に移動させた。
Parts:
- moved U7 0.13 mm to (48.3, -22.7)
- moved U8 0.13 mm to (73.7, -22.7)
- moved U9 0.13 mm to (99.1, -22.7)
Routing:
- net /7seg/KE: track 84.8 -> 0.25 mm
- net /7seg/KF: track 80.5 -> 0.00 mm
- net /KD11: track 66.1 -> 10.2 mm
- net /GND_BNC: track 55.3 -> 10.2 mm, vias 1 -> 0
- net /7seg/KA: track 54.1 -> 94.7 mm
- net /KD20: track 44.3 -> 10.2 mm
- net /SIGNAL: track 33.5 -> 0.00 mm, vias 1 -> 0
- net /7seg/KC: track 54.1 -> 86.9 mm
- net /KD15: track 33.7 -> 5.08 mm
- net /KD24: track 31.4 -> 6.09 mm
- net /KD22: track 34.3 -> 10.2 mm
- net Net-(R29-Pad2): track 33.2 -> 13.3 mm
- net T1VCC: track 82.3 -> 66.0 mm, vias 2 -> 0
- net VCC: track 25.4 -> 10.2 mm
- net /KD13: track 23.0 -> 10.2 mm
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
Commit message: 74HC00系用に，VCC_T1, GND_T1を作成。
母板と74HC00をconnectorで分離したかったため，xxx_T1を作成する必要があった。
Connections:
- J9 pad 1: VCC -> VCC_T1
- J9 pad 2: T1GND -> GND_T1
- Q6 pad 1: T1GND -> GND_T1
- Q7 pad 1: T1GND -> GND_T1
- Q8 pad 1: T1GND -> GND_T1
- R26 pad 2: T1VCC -> VCC_T1
- R30 pad 2: T1VCC -> VCC_T1
- R31 pad 2: T1VCC -> VCC_T1
- R46 pad 1: T1GND -> (no net)
- U4 pad 14: VCC -> VCC_T1
- U4 pad 7: GND -> GND_T1
- U5 pad 14: VCC -> VCC_T1
- U5 pad 7: GND -> GND_T1
- U6 pad 14: VCC -> VCC_T1
- U6 pad 7: GND -> GND_T1
Routing:
- net VCC_T1: track 0.00 -> 5.08 mm
- net T1VCC: track 66.0 -> 61.0 mm

Commit message: TVCC, TGND の壊滅。
Connections:
- C1 pad 1: /TVCC -> VCC
- C2 pad 1: /TVCC -> VCC
- C8 pad 1: /TVCC -> VCC
- D5 pad 2: /TVCC -> VCC
- J1 pad 2: /TVCC -> VCC
- Q10 pad 2: T1VCC -> VCC_T1
- Q11 pad 2: T1VCC -> VCC_T1
- Q12 pad 2: T1VCC -> VCC_T1
- Q13 pad 2: T1VCC -> VCC_T1
- Q14 pad 2: T1VCC -> VCC_T1
- Q3 pad 1: /TVCC -> VCC
- Q9 pad 2: T1VCC -> VCC_T1
- R13 pad 2: /TVCC -> VCC
- R15 pad 2: /TVCC -> VCC
- R2 pad 1: /TVCC -> VCC
- R3 pad 1: /TVCC -> VCC
- R46 pad 1: (no net) -> GND_T1
- SW2 pad 2: /TVCC -> VCC
- U1 pad 14: /TVCC -> VCC
Routing:
- net VCC: track 10.2 -> 76.3 mm
- net /TVCC: track 66.1 -> 0.00 mm
- net VCC_T1: track 5.08 -> 66.0 mm
- net T1VCC: track 61.0 -> 0.00 mm

Commit message: 4色駆使することで，なんとかかんとか7SEG, LEDの配線が完成。
Parts:
- moved J8 74.2 mm to (91.4, -78.7)
- moved Q6 74.2 mm to (68.6, -73.7)
- moved Q7 74.2 mm to (68.6, -68.6)
- moved Q8 74.2 mm to (68.6, -78.7)
- moved R23 74.2 mm to (76.2, -73.7)
- moved R24 74.2 mm to (83.8, -76.2)
- moved R25 74.2 mm to (83.8, -71.1)
- moved R27 74.2 mm to (76.2, -68.6)
- moved R28 74.2 mm to (76.2, -78.7)
- moved R29 74.2 mm to (83.8, -81.3)
- moved U4 74.2 mm to (68.6, -55.9)
- moved R26 74.2 mm to (66.0, -73.7)
- moved R30 74.2 mm to (66.0, -76.2)
- moved R31 74.2 mm to (66.0, -78.7)
- moved J9 57.5 mm to (109.2, -58.4)
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Routing:
- net GND_T1: track 0.00 -> 200.7 mm
- net /7seg/KE: track 0.25 -> 111.6 mm
- net /7seg/KF: track 0.00 -> 99.7 mm
- net /7seg/KDP: track 0.00 -> 83.4 mm
- net Net-(U4-Pad8): track 0.00 -> 62.2 mm
- net VCC_T1: track 66.0 -> 124.5 mm
- net Net-(U4-Pad11): track 0.00 -> 53.3 mm
- net Net-(U4-Pad3): track 0.00 -> 50.5 mm
- net /KD15: track 5.08 -> 54.4 mm
- net Net-(U4-Pad6): track 0.00 -> 47.4 mm
- net /KD13: track 10.2 -> 56.1 mm
- net Net-(R25-Pad2): track 0.00 -> 43.8 mm
- net /KD24: track 6.09 -> 41.2 mm
- net Net-(Q7-Pad2): track 10.2 -> 45.3 mm
- net /7seg/KC: track 86.9 -> 118.4 mm
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
Commit message: Display 部を時計回りに90度回転させて，mother部とくっつけた。
なんとか，2階建てで上手くいきそうな気がする。
Parts:
- moved R29 156.0 mm to (162.6, 53.3), turned to 90 degrees
- moved J8 155.6 mm to (160.0, 61.0), turned to 270 degrees
- moved R28 150.1 mm to (160.0, 45.7), turned to 270 degrees
- moved R24 149.0 mm to (157.5, 53.3), turned to 90 degrees
- moved Q8 148.4 mm to (160.0, 38.1), turned to 270 degrees
- moved R31 148.0 mm to (160.0, 35.6), turned to 90 degrees
- moved R30 144.4 mm to (157.5, 35.6), turned to 90 degrees
- moved U6 143.1 mm to (144.8, 73.7), turned to 180 degrees
- moved R23 143.0 mm to (154.9, 45.7), turned to 270 degrees
- moved R25 142.1 mm to (152.4, 53.3), turned to 90 degrees
- moved Q6 141.2 mm to (154.9, 38.1), turned to 270 degrees
- moved R26 140.8 mm to (154.9, 35.6), turned to 90 degrees
- moved J9 140.5 mm to (139.7, 78.7), turned to 0 degrees
- moved R27 136.0 mm to (149.9, 45.7), turned to 270 degrees
- moved Q7 134.1 mm to (149.9, 38.1), turned to 270 degrees
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Other:
- board size 152.4 x 116.8 mm -> 152.4 x 195.6 mm
- board text added: "Display"
- board text added: "last rotate PAI."

Commit message: 母板部の配線を進めた。Display部を決定したいので，中途半端だがcommit。
Parts:
- moved J10 53.9 mm to (154.9, 167.6), turned to 90 degrees
- moved D1 32.3 mm to (116.8, 119.4), turned to 270 degrees
- moved R1 30.6 mm to (142.2, 116.8)
- moved D2 21.6 mm to (124.5, 119.4), turned to 270 degrees
- moved D3 10.8 mm to (132.1, 119.4), turned to 270 degrees
- moved J9 10.5 mm to (149.9, 76.2), turned to 90 degrees
- moved C4 7.62 mm to (94.0, 157.5)
- turned D4 to 270 degrees
Routing:
- net GND: track 165.8 -> 0.11 mm, vias 1 -> 0
- net VCC: track 76.3 -> 0.18 mm
- net Net-(D1-Pad2): track 22.9 -> 51.9 mm
- net Net-(D2-Pad2): track 27.9 -> 46.8 mm
- net /SIGNAL_BNC: track 0.00 -> 13.8 mm
- net Net-(D3-Pad2): track 17.8 -> 30.0 mm
- net /GND_BNC: track 10.2 -> 0.75 mm
- net GND_T1: track 200.7 -> 192.8 mm
- net Net-(Q1-Pad2): track 20.3 -> 27.9 mm
- net Net-(D1-Pad1): track 27.9 -> 35.6 mm
- net VCC_T1: track 124.5 -> 130.6 mm
- net Net-(J5-Pad8): track 0.00 -> 2.54 mm
- net Net-(J5-Pad7): track 0.00 -> 2.54 mm
- net Net-(J5-Pad6): track 0.00 -> 2.54 mm
- net Net-(J5-Pad5): track 0.00 -> 2.54 mm
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
Commit message: Display部の配線は完成。
Parts:
- moved R38 5.08 mm to (96.5, 83.8)
- moved R40 5.08 mm to (101.6, 83.8)
- moved R39 5.08 mm to (99.1, 83.8)
- moved R41 5.08 mm to (104.1, 83.8)
- moved R42 5.08 mm to (106.7, 83.8)
- moved R43 5.08 mm to (109.2, 83.8)
- moved R44 5.08 mm to (111.8, 83.8)
- moved R45 5.08 mm to (114.3, 83.8)
- moved J7 5.08 mm to (114.3, 94.0)
Routing:
- net /7seg/KA: track 108.5 -> 98.3 mm
- net /7seg/KB: track 63.0 -> 52.8 mm
- net /7seg/KDP: track 83.4 -> 76.8 mm
- net /7seg/KC: track 118.4 -> 113.3 mm
- net /7seg/KE: track 111.6 -> 106.5 mm
- net /7seg/KD: track 68.7 -> 63.6 mm
- net /7seg/KF: track 99.7 -> 94.6 mm
- net /7seg/KG: track 124.5 -> 119.4 mm
