File: pcb/7seg.sch (KiCad schematic (older format))
At the start: 28 parts, among them Q10 2SC1815, Q11 2SC1815, Q12 2SC1815, Q13 2SC1815, Q14 2SC1815, Q9 2SC1815, U7 7seg-2digit-ca, U8 7seg-2digit-ca, U9 7seg-2digit-ca

Commit message: 3Dpackages が表示されるように，旧式の3D modelを使うようにした。
Parts:
- Q10, Q11, Q12, Q13, Q14, Q9: footprint Package_TO_SOT_THT:TO-92_Inline_Wide -> TO_SOT_Packages_THT:TO-92_Inline_Wide
Changed lines of the file:
@@
 F 0 "Q9" H 1450 2750 50  0000 L CNN
 F 1 "2SC1815" H 1350 2850 50  0000 L CNN
-F 2 "Package_TO_SOT_THT:TO-92_Inline_Wide" H 1800 2575 50  0001 L CIN
+F 2 "TO_SOT_Packages_THT:TO-92_Inline_Wide" H 1800 2575 50  0001 L CIN
 F 3 "" H 1600 2650 50  0001 L CNN
 	1    1600 2650
@@
 F 0 "Q10" H 1850 2850 50  0000 L CNN
 F 1 "2SC1815" H 1750 2950 50  0000 L CNN
-F 2 "Package_TO_SOT_THT:TO-92_Inline_Wide" H 2200 2675 50  0001 L CIN
+F 2 "TO_SOT_Packages_THT:TO-92_Inline_Wide" H 2200 2675 50  0001 L CIN
 F 3 "" H 2000 2750 50  0001 L CNN
 	1    2000 2750
@@
 F 0 "Q11" H 2250 2950 50  0000 L CNN
 F 1 "2SC1815" H 2150 3050 50  0000 L CNN
-F 2 "Package_TO_SOT_THT:TO-92_Inline_Wide" H 2600 2775 50  0001 L CIN
+F 2 "TO_SOT_Packages_THT:TO-92_Inline_Wide" H 2600 2775 50  0001 L CIN
 F 3 "" H 2400 2850 50  0001 L CNN
 	1    2400 2850
@@
 F 0 "Q12" H 2650 3050 50  0000 L CNN
 F 1 "2SC1815" H 2550 3150 50  0000 L CNN
-F 2 "Package_TO_SOT_THT:TO-92_Inline_Wide" H 3000 2875 50  0001 L CIN
+F 2 "TO_SOT_Packages_THT:TO-92_Inline_Wide" H 3000 2875 50  0001 L CIN
 F 3 "" H 2800 2950 50  0001 L CNN
 	1    2800 2950
@@
 F 0 "Q13" H 3050 3150 50  0000 L CNN
 F 1 "2SC1815" H 2950 3250 50  0000 L CNN
-F 2 "Package_TO_SOT_THT:TO-92_Inline_Wide" H 3400 2975 50  0001 L CIN
+F 2 "TO_SOT_Packages_THT:TO-92_Inline_Wide" H 3400 2975 50  0001 L CIN
 F 3 "" H 3200 3050 50  0001 L CNN
 	1    3200 3050
@@
 F 0 "Q14" H 3450 3250 50  0000 L CNN
 F 1 "2SC1815" H 3350 3350 50  0000 L CNN
-F 2 "Package_TO_SOT_THT:TO-92_Inline_Wide" H 3800 3075 50  0001 L CIN
+F 2 "TO_SOT_Packages_THT:TO-92_Inline_Wide" H 3800 3075 50  0001 L CIN
 F 3 "" H 3600 3150 50  0001 L CNN
 	1    3600 3150

Commit message: transistor には，CvPcbをやり直した。
Parts:
- Q10, Q11, Q12, Q13, Q14, Q9: footprint TO_SOT_Packages_THT:TO-92_Inline_Wide -> Package_TO_SOT_THT:TO-92_Inline_Wide
Changed lines of the file:
@@
 F 0 "Q9" H 1450 2750 50  0000 L CNN
 F 1 "2SC1815" H 1350 2850 50  0000 L CNN
-F 2 "TO_SOT_Packages_THT:TO-92_Inline_Wide" H 1800 2575 50  0001 L CIN
+F 2 "Package_TO_SOT_THT:TO-92_Inline_Wide" H 1800 2575 50  0001 L CIN
 F 3 "" H 1600 2650 50  0001 L CNN
 	1    1600 2650
@@
 F 0 "Q10" H 1850 2850 50  0000 L CNN
 F 1 "2SC1815" H 1750 2950 50  0000 L CNN
-F 2 "TO_SOT_Packages_THT:TO-92_Inline_Wide" H 2200 2675 50  0001 L CIN
+F 2 "Package_TO_SOT_THT:TO-92_Inline_Wide" H 2200 2675 50  0001 L CIN
 F 3 "" H 2000 2750 50  0001 L CNN
 	1    2000 2750
@@
 F 0 "Q11" H 2250 2950 50  0000 L CNN
 F 1 "2SC1815" H 2150 3050 50  0000 L CNN
-F 2 "TO_SOT_Packages_THT:TO-92_Inline_Wide" H 2600 2775 50  0001 L CIN
+F 2 "Package_TO_SOT_THT:TO-92_Inline_Wide" H 2600 2775 50  0001 L CIN
 F 3 "" H 2400 2850 50  0001 L CNN
 	1    2400 2850
@@
 F 0 "Q12" H 2650 3050 50  0000 L CNN
 F 1 "2SC1815" H 2550 3150 50  0000 L CNN
-F 2 "TO_SOT_Packages_THT:TO-92_Inline_Wide" H 3000 2875 50  0001 L CIN
+F 2 "Package_TO_SOT_THT:TO-92_Inline_Wide" H 3000 2875 50  0001 L CIN
 F 3 "" H 2800 2950 50  0001 L CNN
 	1    2800 2950
@@
 F 0 "Q13" H 3050 3150 50  0000 L CNN
 F 1 "2SC1815" H 2950 3250 50  0000 L CNN
-F 2 "TO_SOT_Packages_THT:TO-92_Inline_Wide" H 3400 2975 50  0001 L CIN
+F 2 "Package_TO_SOT_THT:TO-92_Inline_Wide" H 3400 2975 50  0001 L CIN
 F 3 "" H 3200 3050 50  0001 L CNN
 	1    3200 3050
@@
 F 0 "Q14" H 3450 3250 50  0000 L CNN
 F 1 "2SC1815" H 3350 3350 50  0000 L CNN
-F 2 "TO_SOT_Packages_THT:TO-92_Inline_Wide" H 3800 3075 50  0001 L CIN
+F 2 "Package_TO_SOT_THT:TO-92_Inline_Wide" H 3800 3075 50  0001 L CIN
 F 3 "" H 3600 3150 50  0001 L CNN
 	1    3600 3150
