File: pcb/3in8out.sch (KiCad schematic (older format))
At the start: 15 parts, among them Q6 CSC388A, Q7 CSC388A, Q8 CSC388A, U4 74HC00, U5 74HC00, U6 74HC00

Commit message: 3Dpackages が表示されるように，旧式の3D modelを使うようにした。
Parts:
- Q6, Q7, Q8: footprint Package_TO_SOT_THT:TO-92_Inline_Wide -> TO_SOT_Packages_THT:TO-92_Inline_Wide
- U4, U5, U6: footprint Housings_DIP:DIP-14_W7.62mm -> Package_DIP:DIP-14_W7.62mm
Changed lines of the file:
@@
 F 0 "U4" H 5350 1700 50  0000 C CNN
 F 1 "74HC00" H 5350 1550 50  0000 C CNN
-F 2 "Housings_DIP:DIP-14_W7.62mm" H 5350 1650 50  0001 C CNN
+F 2 "Package_DIP:DIP-14_W7.62mm" H 5350 1650 50  0001 C CNN
 F 3 "" H 5350 1650 50  0001 C CNN
 	1    5350 1650
@@
 F 0 "U4" H 5350 2250 50  0000 C CNN
 F 1 "74HC00" H 5350 2100 50  0000 C CNN
-F 2 "Housings_DIP:DIP-14_W7.62mm" H 5350 2200 50  0001 C CNN
+F 2 "Package_DIP:DIP-14_W7.62mm" H 5350 2200 50  0001 C CNN
 F 3 "" H 5350 2200 50  0001 C CNN
 	2    5350 2200
@@
 F 0 "U4" H 5350 2800 50  0000 C CNN
 F 1 "74HC00" H 5350 2650 50  0000 C CNN
-F 2 "Housings_DIP:DIP-14_W7.62mm" H 5350 2750 50  0001 C CNN
+F 2 "Package_DIP:DIP-14_W7.62mm" H 5350 2750 50  0001 C CNN
 F 3 "" H 5350 2750 50  0001 C CNN
 	3    5350 2750
@@
 F 0 "U4" H 5350 3350 50  0000 C CNN
 F 1 "74HC00" H 5350 3200 50  0000 C CNN
-F 2 "Housings_DIP:DIP-14_W7.62mm" H 5350 3300 50  0001 C CNN
+F 2 "Package_DIP:DIP-14_W7.62mm" H 5350 3300 50  0001 C CNN
 F 3 "" H 5350 3300 50  0001 C CNN
 	4    5350 3300
@@
 F 0 "U6" H 7450 1800 50  0000 C CNN
 F 1 "74HC00" H 7450 1650 50  0000 C CNN
-F 2 "Housings_DIP:DIP-14_W7.62mm" H 7450 1750 50  0001 C CNN
+F 2 "Package_DIP:DIP-14_W7.62mm" H 7450 1750 50  0001 C CNN
 F 3 "" H 7450 1750 50  0001 C CNN
 	1    7450 1750
@@
 F 0 "U6" H 7450 2350 50  0000 C CNN
 F 1 "74HC00" H 7450 2200 50  0000 C CNN
-F 2 "Housings_DIP:DIP-14_W7.62mm" H 7450 2300 50  0001 C CNN
+F 2 "Package_DIP:DIP-14_W7.62mm" H 7450 2300 50  0001 C CNN
 F 3 "" H 7450 2300 50  0001 C CNN
 	2    7450 2300
@@
 F 0 "U6" H 7450 2900 50  0000 C CNN
 F 1 "74HC00" H 7450 2750 50  0000 C CNN
-F 2 "Housings_DIP:DIP-14_W7.62mm" H 7450 2850 50  0001 C CNN
+F 2 "Package_DIP:DIP-14_W7.62mm" H 7450 2850 50  0001 C CNN
 F 3 "" H 7450 2850 50  0001 C CNN
 	3    7450 2850
@@
 F 0 "U6" H 7450 3450 50  0000 C CNN
 F 1 "74HC00" H 7450 3300 50  0000 C CNN
-F 2 "Housings_DIP:DIP-14_W7.62mm" H 7450 3400 50  0001 C CNN
+F 2 "Package_DIP:DIP-14_W7.62mm" H 7450 3400 50  0001 C CNN
 F 3 "" H 7450 3400 50  0001 C CNN
 	4    7450 3400
@@
 F 0 "U5" H 7400 4200 50  0000 C CNN
 F 1 "74HC00" H 7400 4050 50  0000 C CNN
-F 2 "Housings_DIP:DIP-14_W7.62mm" H 7400 4150 50  0001 C CNN
+F 2 "Package_DIP:DIP-14_W7.62mm" H 7400 4150 50  0001 C CNN
 F 3 "" H 7400 4150 50  0001 C CNN
 	1    7400 4150
@@
 F 0 "U5" H 7400 4750 50  0000 C CNN
 F 1 "74HC00" H 7400 4600 50  0000 C CNN
-F 2 "Housings_DIP:DIP-14_W7.62mm" H 7400 4700 50  0001 C CNN
+F 2 "Package_DIP:DIP-14_W7.62mm" H 7400 4700 50  0001 C CNN
 F 3 "" H 7400 4700 50  0001 C CNN
 	2    7400 4700
@@
 F 0 "U5" H 7400 5300 50  0000 C CNN
 F 1 "74HC00" H 7400 5150 50  0000 C CNN
-F 2 "Housings_DIP:DIP-14_W7.62mm" H 7400 5250 50  0001 C CNN
+F 2 "Package_DIP:DIP-14_W7.62mm" H 7400 5250 50  0001 C CNN
 F 3 "" H 7400 5250 50  0001 C CNN
 	3    7400 5250
@@
 F 0 "U5" H 7400 5850 50  0000 C CNN
 F 1 "74HC00" H 7400 5700 50  0000 C CNN
-F 2 "Housings_DIP:DIP-14_W7.62mm" H 7400 5800 50  0001 C CNN
+F 2 "Package_DIP:DIP-14_W7.62mm" H 7400 5800 50  0001 C CNN
 F 3 "" H 7400 5800 50  0001 C CNN
 	4    7400 5800
@@
 F 0 "Q8" H 3700 1950 50  0000 L CNN
 F 1 "CSC388A" V 3950 1650 50  0000 L CNN
-F 2 "Package_TO_SOT_THT:TO-92_Inline_Wide" H 3950 1725 50  0001 L CIN
+F 2 "TO_SOT_Packages_THT:TO-92_Inline_Wide" H 3950 1725 50  0001 L CIN
 F 3 "" H 3750 1800 50  0001 L CNN
 	1    3750 1800
@@
 F 0 "Q6" H 3350 2900 50  0000 L CNN
 F 1 "CSC388A" V 3600 2600 50  0000 L CNN
-F 2 "Package_TO_SOT_THT:TO-92_Inline_Wide" H 3600 2675 50  0001 L CIN
+F 2 "TO_SOT_Packages_THT:TO-92_Inline_Wide" H 3600 2675 50  0001 L CIN
 F 3 "" H 3400 2750 50  0001 L CNN
 	1    3400 2750
@@
 F 0 "Q7" H 3350 4850 50  0000 L CNN
 F 1 "CSC388A" V 3600 4550 50  0000 L CNN
-F 2 "Package_TO_SOT_THT:TO-92_Inline_Wide" H 3600 4625 50  0001 L CIN
+F 2 "TO_SOT_Packages_THT:TO-92_Inline_Wide" H 3600 4625 50  0001 L CIN
 F 3 "" H 3400 4700 50  0001 L CNN
 	1    3400 4700

Commit message: KiCad 5.0 change some files.
Parts:
- Q6, Q7, Q8: symbol CSC388A -> freq-counter-rescue:CSC388A
- R23, R24, R25, R26, R27, R28, R29, R30, R31: symbol R -> freq-counter-rescue:R
- U4, U5, U6: symbol 74HC00 -> freq-counter-rescue:74HC00
Changed lines of the file:
@@
-EESchema Schematic File Version 2
-LIBS:7seg-4digit
-LIBS:power
-LIBS:device
-LIBS:switches
-LIBS:relays
-LIBS:motors
-LIBS:transistors
-LIBS:conn
-LIBS:linear
-LIBS:regul
-LIBS:74xx
-LIBS:cmos4000
-LIBS:adc-dac
-LIBS:memory
-LIBS:xilinx
-LIBS:microcontrollers
-LIBS:dsp
-LIBS:microchip
-LIBS:analog_switches
-LIBS:motorola
-LIBS:texas
-LIBS:intel
-LIBS:audio
-LIBS:interface
-LIBS:digital-audio
-LIBS:philips
-LIBS:display
-LIBS:cypress
-LIBS:siliconi
-LIBS:opto
-LIBS:atmel
-LIBS:contrib
-LIBS:valves
+EESchema Schematic File Version 4
 LIBS:freq-counter-cache
-EELAYER 25 0
+EELAYER 26 0
 EELAYER END
 $Descr A4 11693 8268
@@
 $EndDescr
 $Comp
-L 74HC00 U4
+L freq-counter-rescue:74HC00 U4
 U 1 1 5A10DC2D
 P 5350 1650
@@
 $EndComp
 $Comp
-L 74HC00 U4
+L freq-counter-rescue:74HC00 U4
 U 2 1 5A10DC34
 P 5350 2200
@@
 $EndComp
 $Comp
-L 74HC00 U4
+L freq-counter-rescue:74HC00 U4
 U 3 1 5A10DC3B
 P 5350 2750
@@
 $EndComp
 $Comp
-L 74HC00 U4
+L freq-counter-rescue:74HC00 U4
 U 4 1 5A10DC42
 P 5350 3300
@@
 $EndComp
 $Comp
-L 74HC00 U6
+L freq-counter-rescue:74HC00 U6
 U 1 1 5A10DC49
 P 7450 1750
@@
 $EndComp
 $Comp
-L 74HC00 U6
+L freq-counter-rescue:74HC00 U6
 U 2 1 5A10DC50
 P 7450 2300
@@
 $EndComp
 $Comp
-L 74HC00 U6
+L freq-counter-rescue:74HC00 U6
 U 3 1 5A10DC57
 P 7450 2850
@@
 $EndComp
 $Comp
-L 74HC00 U6
+L freq-counter-rescue:74HC00 U6
 U 4 1 5A10DC5E
 P 7450 3400
@@
 $EndComp
 $Comp
-L 74HC00 U5
+L freq-counter-rescue:74HC00 U5
 U 1 1 5A10DC65
 P 7400 4150
@@
 $EndComp
 $Comp
-L 74HC00 U5
+L freq-counter-rescue:74HC00 U5
 U 2 1 5A10DC6C
 P 7400 4700
@@
 $EndComp
 $Comp
-L 74HC00 U5
+L freq-counter-rescue:74HC00 U5
 U 3 1 5A10DC73
 P 7400 5250
@@
 $EndComp
 $Comp
-L 74HC00 U5
+L freq-counter-rescue:74HC00 U5
 U 4 1 5A10DC7A
 P 7400 5800
@@
 $EndComp
 $Comp
-L CSC388A Q8
+L freq-counter-rescue:CSC388A Q8
 U 1 1 5A10DC81
 P 3750 1800
@@
 $EndComp
 $Comp
-L R R28
+L freq-counter-rescue:R R28
 U 1 1 5A10DC88
 P 3250 1800
@@
 $EndComp
 $Comp
-L R R31
+L freq-counter-rescue:R R31
 U 1 1 5A10DC8F
 P 3850 1300
@@
 $EndComp
 $Comp
-L R R29
+L freq-counter-rescue:R R29
 U 1 1 5A10DC96
 P 3250 2100
@@
 $EndComp
 $Comp
-L CSC388A Q6
+L freq-counter-rescue:CSC388A Q6
 U 1 1 5A10DC9D
 P 3400 2750
@@
 $EndComp
 $Comp
-L R R23
+L freq-counter-rescue:R R23
 U 1 1 5A10DCA4
 P 2950 2750
@@
 $EndComp
 $Comp
-L R R30
+L freq-counter-rescue:R R30
 U 1 1 5A10DCAB
 P 3500 1300
@@
 $EndComp
 $Comp
-L R R24
+L freq-counter-rescue:R R24
 U 1 1 5A10DCB2
 P 2950 3200
@@
 $EndComp
 $Comp
-L CSC388A Q7
+L freq-counter-rescue:CSC388A Q7
 U 1 1 5A10DCE5
 P 3400 4700
@@
 $EndComp
 $Comp
-L R R27
+L freq-counter-rescue:R R27
 U 1 1 5A10DCEC
 P 2950 4700
@@
 $EndComp
 $Comp
-L R R25
+L freq-counter-rescue:R R25
 U 1 1 5A10DCF3
 P 2950 3600
@@
 $EndComp
 $Comp
-L R R26
+L freq-counter-rescue:R R26
 U 1 1 5A10DD03
 P 2950 4250
